Commit message: changing body build function

File: recursive_body_test.urdf (robot description, URDF)
Before this commit: robot robot, 11 links, 10 joints
Links:
- link 0: geometry collision box size=0.976935060891263 0.5961857580704077 0.46746389529285814; visual box size=0.976935060891263 0.5961857580704077 0.46746389529285814
- link 1: geometry collision box size=0.9799070242381127 0.7038721641123848 0.20530203832510782; visual box size=0.9799070242381127 0.7038721641123848 0.20530203832510782
- link 10: geometry collision box size=0.9136751067579685 0.8995819010116815 0.3305040818956976; visual box size=0.9136751067579685 0.8995819010116815 0.3305040818956976
- link 2: geometry collision box size=0.9598644003046919 0.7147171463021396 0.5076992357440557; visual box size=0.9598644003046919 0.7147171463021396 0.5076992357440557
- link 3: geometry collision box size=0.3405262867409823 0.25709766006961154 0.4693655576513629; visual box size=0.3405262867409823 0.25709766006961154 0.4693655576513629
- link 4: geometry collision box size=0.9436783459008433 0.9381947555759376 0.18116934923550862; visual box size=0.9436783459008433 0.9381947555759376 0.18116934923550862
- link 5: geometry collision box size=0.706853414963293 0.5367660821898774 0.2750923768330873; visual box size=0.706853414963293 0.5367660821898774 0.2750923768330873
- link 6: geometry collision box size=0.6216894307044214 0.33900713284589507 0.26139621087047493; visual box size=0.6216894307044214 0.33900713284589507 0.26139621087047493
- link 7: geometry collision box size=0.5248636858205162 0.888543975175575 0.5235752481678471; visual box size=0.5248636858205162 0.888543975175575 0.5235752481678471
- link 8: geometry collision box size=0.7446781712666404 0.2789744931071074 0.4997867331889747; visual box size=0.7446781712666404 0.2789744931071074 0.4997867331889747
- link 9: geometry collision box size=0.9426034922729505 0.8060273752894318 0.5848762315014768; visual box size=0.9426034922729505 0.8060273752894318 0.5848762315014768
Joints:
- joint 0_1: origin xyz=0.5610301526762972 0.0 0.0 rpy=0 0 0 -> xyz=0.976935060891263 0.0 2.0 rpy=0 0 0
- joint 1_2: origin xyz=0.21787049445972728 0.0 0.0 rpy=0 0 0 -> xyz=0.9799070242381127 0.0 0.0 rpy=0 0 0
- joint 2_3: origin xyz=0.36907214464235755 0.0 0.0 rpy=0 0 0 -> xyz=0.9598644003046919 0.0 0.0 rpy=0 0 0
- joint 3_4: origin xyz=1.2780648849068668 0.0 0.0 rpy=0 0 0 -> xyz=0.3405262867409823 0.0 0.0 rpy=0 0 0
- joint 4_5: origin xyz=0.42171848376181487 0.0 0.0 rpy=0 0 0 -> xyz=0.9436783459008433 0.0 0.0 rpy=0 0 0
- joint 5_6: origin xyz=1.0485576125161957 0.0 0.0 rpy=0 0 0 -> xyz=0.706853414963293 0.0 0.0 rpy=0 0 0
- joint 6_7: origin xyz=0.29230152316736047 0.0 0.0 rpy=0 0 0 -> xyz=0.6216894307044214 0.0 0.0 rpy=0 0 0
- joint 7_8: origin xyz=0.5247824523147964 0.0 0.0 rpy=0 0 0 -> xyz=0.5248636858205162 0.0 0.0 rpy=0 0 0
- joint 8_9: origin xyz=1.3857581573584188 0.0 0.0 rpy=0 0 0 -> xyz=0.7446781712666404 0.0 0.0 rpy=0 0 0
- joint 9_10: origin xyz=0.6121689359574695 0.0 0.0 rpy=0 0 0 -> xyz=0.9426034922729505 0.0 0.0 rpy=0 0 0

Commit message: color working

File: recursive_body_test.urdf (robot description, URDF)
Before this commit: robot robot, 11 links, 10 joints
Links:
- link 0: geometry collision box size=0.2708415955312511 0.27586075261945137 0.10646559581195744; visual box size=0.2708415955312511 0.27586075261945137 0.10646559581195744
- link 1: geometry collision box size=0.40111113440553514 0.34245967285882106 0.4217623888965252; visual box size=0.40111113440553514 0.34245967285882106 0.4217623888965252
- link 10: geometry collision box size=0.7788989703641653 0.7858508731999059 0.45120016396007734; visual box size=0.7788989703641653 0.7858508731999059 0.45120016396007734
- link 2: geometry collision box size=0.8260421018610506 0.2614746870539584 0.36586881974017327; visual box size=0.8260421018610506 0.2614746870539584 0.36586881974017327
- link 3: geometry collision box size=0.6588268006588816 0.6962518744921455 0.24881658857014596; visual box size=0.6588268006588816 0.6962518744921455 0.24881658857014596
- link 4: geometry collision box size=0.3682613056482067 0.38922174356105477 0.31574480704916175; visual box size=0.3682613056482067 0.38922174356105477 0.31574480704916175
- link 5: geometry collision box size=0.5395523927167667 0.3563313203760233 0.25702366433140234; visual box size=0.5395523927167667 0.3563313203760233 0.25702366433140234
- link 6: geometry collision box size=0.8383926479067072 0.8942903059483329 0.41929187058874207; visual box size=0.8383926479067072 0.8942903059483329 0.41929187058874207
- link 7: geometry collision box size=0.5708309345006501 0.79396190256298 0.5844738723448035; visual box size=0.5708309345006501 0.79396190256298 0.5844738723448035
- link 8: geometry collision box size=0.7817980107709854 0.2486558359958343 0.5678336998781436; visual box size=0.7817980107709854 0.2486558359958343 0.5678336998781436
- link 9: geometry collision box size=0.604188113766656 0.25969668040022875 0.49580353088271645; visual box size=0.604188113766656 0.25969668040022875 0.49580353088271645
Joints:
- joint 0_1: origin xyz=0.976935060891263 0.0 2.0 rpy=0 0 0 -> xyz=0.2708415955312511 0.0 2.0 rpy=0 0 0
- joint 1_2: origin xyz=0.9799070242381127 0.0 0.0 rpy=0 0 0 -> xyz=0.40111113440553514 0.0 0.0 rpy=0 0 0
- joint 2_3: origin xyz=0.9598644003046919 0.0 0.0 rpy=0 0 0 -> xyz=0.8260421018610506 0.0 0.0 rpy=0 0 0
- joint 3_4: origin xyz=0.3405262867409823 0.0 0.0 rpy=0 0 0 -> xyz=0.6588268006588816 0.0 0.0 rpy=0 0 0
- joint 4_5: origin xyz=0.9436783459008433 0.0 0.0 rpy=0 0 0 -> xyz=0.3682613056482067 0.0 0.0 rpy=0 0 0
- joint 5_6: origin xyz=0.706853414963293 0.0 0.0 rpy=0 0 0 -> xyz=0.5395523927167667 0.0 0.0 rpy=0 0 0
- joint 6_7: origin xyz=0.6216894307044214 0.0 0.0 rpy=0 0 0 -> xyz=0.8383926479067072 0.0 0.0 rpy=0 0 0
- joint 7_8: origin xyz=0.5248636858205162 0.0 0.0 rpy=0 0 0 -> xyz=0.5708309345006501 0.0 0.0 rpy=0 0 0
- joint 8_9: origin xyz=0.7446781712666404 0.0 0.0 rpy=0 0 0 -> xyz=0.7817980107709854 0.0 0.0 rpy=0 0 0
- joint 9_10: origin xyz=0.9426034922729505 0.0 0.0 rpy=0 0 0 -> xyz=0.604188113766656 0.0 0.0 rpy=0 0 0
